Commit message: Lab robot: real body shape with the LiDAR on the top deck and the camera on the middle deck; demo videos follow the README steps
- tc70045e_sim: lab_robot.urdf.xacro uses the robot's real body, wheel, LiDAR and camera meshes (meshes/lab_robot,
  BSD-3-Clause); the sensors now sit on the body (LiDAR scan plane 18.1 cm, camera 10.9 cm) instead of floating
  above it. Frame names, topics and wheel kinematics are unchanged.
- lab.world: default Gazebo view shows both rooms.
- tools/demo: week04-08 demo scripts rewritten to follow each README and lecture step by step (A1..An, the
  activity, solution last); commands stay on screen; long drives played faster; gzview.py sets the Gazebo view.
- Week 4 README: LiDAR slice 18 cm; Week 1 TF example updated; Weeks 6-7: Assessment 1 (50 %) due in Week 7.

File: docker/tc70045e_sim/urdf/lab_robot.urdf.xacro (robot description, xacro)
@@ -19,23 +19,33 @@
   <xacro:arg name="camera_height" default="480"/>
   <xacro:property name="p" value="$(arg prefix)"/>
-  <!-- Geometry used in the lectures: r = 37.5 mm, lx = 95 mm, ly = 85 mm (lx + ly = 0.18 m) -->
+  <!-- Wheel geometry used in the lectures and by the wheel_odometry node: r = 37.5 mm, lx = 95 mm, ly = 85 mm
+       (lx + ly = 0.18 m). The body below is the lab robot's real shape: three decks on brass standoffs, the
+       LiDAR on the top deck, the depth camera on the middle deck, four mecanum wheels. -->
   <xacro:property name="r" value="0.0375"/>
   <xacro:property name="lx" value="0.095"/>
   <xacro:property name="ly" value="0.085"/>
-  <xacro:property name="body_l" value="0.30"/>
-  <xacro:property name="body_w" value="0.20"/>
-  <xacro:property name="body_h" value="0.08"/>
+  <!-- Mounting geometry of the real robot (metres). base_link sits 71.4 mm above the floor (wheel axle + 38.9 mm). -->
+  <xacro:property name="base_z" value="0.0714"/>
+  <xacro:property name="mesh_z" value="-0.0064"/>      <!-- chassis meshes are drawn 6.4 mm below base_link -->
+  <xacro:property name="wheel_x" value="0.080"/>
+  <xacro:property name="wheel_y" value="0.0845"/>
+  <xacro:property name="wheel_z" value="-0.0389"/>
+  <xacro:property name="mesh" value="file://$(find tc70045e_sim)/meshes/lab_robot"/>
   <link name="${p}base_footprint"/>
   <link name="${p}base_link">
     <visual>
-      <geometry><box size="${body_l} ${body_w} ${body_h}"/></geometry>
-      <material name="body"><color rgba="0.20 0.25 0.35 1"/></material>
+      <origin xyz="0 0 ${mesh_z}" rpy="0 0 0"/>
+      <geometry><mesh filename="${mesh}/body.obj"/></geometry>
     </visual>
+    <!-- One box around the decks, from 2 mm above the floor to the top deck (below the LiDAR's scan plane,
+         so the LiDAR never sees its own robot) -->
     <collision>
-      <geometry><box size="${body_l} ${body_w} ${body_h}"/></geometry>
+      <origin xyz="0.003 0 -0.0019" rpy="0 0 0"/>
+      <geometry><box size="0.228 0.14 0.135"/></geometry>
     </collision>
     <inertial>
+      <origin xyz="0.003 0 -0.0019" rpy="0 0 0"/>
       <mass value="3.0"/>
-      <inertia ixx="0.0117" ixy="0" ixz="0" iyy="0.0241" iyz="0" izz="0.0325"/>
+      <inertia ixx="0.0094" ixy="0" ixz="0" iyy="0.0176" iyz="0" izz="0.0179"/>
     </inertial>
   </link>
@@ -43,8 +53,7 @@
     <parent link="${p}base_footprint"/>
     <child link="${p}base_link"/>
-    <origin xyz="0 0 ${body_h/2 + 0.002}" rpy="0 0 0"/>
+    <origin xyz="0 0 ${base_z}" rpy="0 0 0"/>
   </joint>
   <gazebo reference="${p}base_link">
-    <material>Gazebo/DarkGrey</material>
     <mu1>0.0</mu1>
     <mu2>0.0</mu2>
@@ -54,7 +63,5 @@
     <link name="${p}wheel_${name}_link">
       <visual>
-        <origin xyz="0 0 0" rpy="${pi/2} 0 0"/>
-        <geometry><cylinder radius="${r}" length="0.035"/></geometry>
-        <material name="wheel"><color rgba="0.05 0.05 0.05 1"/></material>
+        <geometry><mesh filename="${mesh}/wheel_${name}.obj"/></geometry>
       </visual>
       <inertial>
@@ -66,21 +73,17 @@
       <parent link="${p}base_link"/>
       <child link="${p}wheel_${name}_link"/>
-      <origin xyz="${x} ${y} ${r - body_h/2 - 0.002}" rpy="0 0 0"/>
+      <origin xyz="${x} ${y} ${wheel_z}" rpy="0 0 0"/>
     </joint>
-    <gazebo reference="${p}wheel_${name}_link"><material>Gazebo/Black</material></gazebo>
   </xacro:macro>
-  <xacro:wheel name="fl" x="${lx}" y="${ly + 0.02}"/>
-  <xacro:wheel name="fr" x="${lx}" y="${-ly - 0.02}"/>
-  <xacro:wheel name="rl" x="${-lx}" y="${ly + 0.02}"/>
-  <xacro:wheel name="rr" x="${-lx}" y="${-ly - 0.02}"/>
-  <!-- 2D LiDAR -->
+  <xacro:wheel name="fl" x="${wheel_x}" y="${wheel_y}"/>
+  <xacro:wheel name="fr" x="${wheel_x}" y="${-wheel_y}"/>
+  <xacro:wheel name="rl" x="${-wheel_x}" y="${wheel_y}"/>
+  <xacro:wheel name="rr" x="${-wheel_x}" y="${-wheel_y}"/>
+  <!-- 2D LiDAR on the top deck: scan plane 18.1 cm above the floor -->
   <link name="${p}laser_link">
     <visual>
-      <geometry><cylinder radius="0.035" length="0.04"/></geometry>
-      <material name="lidar"><color rgba="0.1 0.1 0.1 1"/></material>
+      <origin xyz="0 0 ${mesh_z}" rpy="0 0 ${pi}"/>
+      <geometry><mesh filename="${mesh}/lidar.obj"/></geometry>
     </visual>
-    <collision>
-      <geometry><cylinder radius="0.035" length="0.04"/></geometry>
-    </collision>
     <inertial>
       <mass value="0.17"/>
@@ -91,8 +94,7 @@
     <parent link="${p}base_link"/>
     <child link="${p}laser_link"/>
-    <origin xyz="0.02 0 ${body_h/2 + 0.06}" rpy="0 0 0"/>
+    <origin xyz="0.043 0 0.110" rpy="0 0 0"/>
   </joint>
   <gazebo reference="${p}laser_link">
-    <material>Gazebo/FlatBlack</material>
     <sensor type="ray" name="lidar">
       <pose>0 0 0 0 0 0</pose>
@@ -184,6 +186,6 @@
   <link name="${p}camera_link">
     <visual>
-      <geometry><box size="0.026 0.124 0.029"/></geometry>
-      <material name="cam"><color rgba="0.6 0.6 0.6 1"/></material>
+      <origin xyz="0 0 ${mesh_z}" rpy="0 0 0"/>
+      <geometry><mesh filename="${mesh}/camera.obj"/></geometry>
     </visual>
     <inertial>
@@ -192,8 +194,9 @@
     </inertial>
   </link>
+  <!-- Depth camera on its bracket on the middle deck: lens 10.9 cm above the floor, looking straight ahead -->
   <joint name="${p}camera_joint" type="fixed">
     <parent link="${p}base_link"/>
     <child link="${p}camera_link"/>
-    <origin xyz="0.14 0 ${body_h/2 + 0.05}" rpy="0 0 0"/>
+    <origin xyz="0.057 0 0.0376" rpy="0 0 0"/>
   </joint>
   <link name="${p}camera_color_optical_frame"/>
@@ -205,5 +208,4 @@
   <xacro:if value="$(arg camera)">
     <gazebo reference="${p}camera_link">
-      <material>Gazebo/Grey</material>
       <sensor name="rgbd" type="depth">
         <always_on>true</always_on>
